Commit message: VALOR PLATO 1

File: ixnaminki_description/urdf/ixnaminki_des.urdf.xacro (robot description, xacro)
@@ -2,4 +2,6 @@
 <robot xmlns:xacro="http://www.ros.org/wiki/xacro" name="ixnaminki_olinki">
     <xacro:property name="PI" value="3.14159265359" />
+    <xacro:property name="effort" value="30.0" />
+    <xacro:property name="velocity" value="10.0" />
     <link name="world"/>
     <link name="base_link">
@@ -59,4 +61,12 @@
         </visual>
     </link>
+    <link name="01_Placa">
+        <visual>
+            <origin xyz="-0.43 1.015 0.55" rpy="1.570795 ${PI} 0.0"/>
+            <geometry>
+                <mesh filename="package://ixnaminki_description/meshes/FLIPPER_ASSY/Placa.STL" scale="0.004 0.004 0.004"/>
+            </geometry>
+        </visual>
+    </link>
     <joint name="virtual_joint" type="fixed">
         <parent link="world"/>
@@ -94,3 +104,11 @@
         <child link="04_PlateSprocket"/>
     </joint>
+    <joint name ="joint_7" type="revolute">
+        <parent link="02_EjePrincipal2"/>
+        <child link = "01_Placa"/>
+        <origin xyz="0.0 0.0 0.0"/>
+        <axis xyz="0 1 0"/>
+        <limit lower="-1.570795" upper="1.570795"
+               effort="${effort}" velocity="${velocity}"/>
+    </joint>
 </robot>

Commit message: Act6ualizando

File: ixnaminki_description/urdf/ixnaminki_des.urdf.xacro (robot description, xacro)
@@ -63,7 +63,47 @@
     <link name="01_Placa">
         <visual>
-            <origin xyz="-0.43 1.015 0.55" rpy="1.570795 ${PI} 0.0"/>
+            <origin xyz="0.26 0.015 0.27" rpy="1.570795 ${PI} 0.0"/>
             <geometry>
                 <mesh filename="package://ixnaminki_description/meshes/FLIPPER_ASSY/Placa.STL" scale="0.004 0.004 0.004"/>
+            </geometry>
+        </visual>
+    </link>
+    <link name="02_Placa">
+        <visual>
+            <origin xyz="0.26 -0.015 0.27" rpy="1.570795 ${PI} 0.0"/>
+            <geometry>
+                <mesh filename="package://ixnaminki_description/meshes/FLIPPER_ASSY/Placa.STL" scale="0.004 0.004 0.004"/>
+            </geometry>
+        </visual>
+    </link>
+    <link name="03_Placa">
+        <visual>
+            <origin xyz="-0.26 0.015 -0.27" rpy="1.570795 0.0 0.0"/>
+            <geometry>
+                <mesh filename="package://ixnaminki_description/meshes/FLIPPER_ASSY/Placa.STL" scale="0.004 0.004 0.004"/>
+            </geometry>
+        </visual>
+    </link>
+    <link name="04_Placa">
+        <visual>
+            <origin xyz="-0.26 -0.015 -0.27" rpy="1.570795 0.0 0.0"/>
+            <geometry>
+                <mesh filename="package://ixnaminki_description/meshes/FLIPPER_ASSY/Placa.STL" scale="0.004 0.004 0.004"/>
+            </geometry>
+        </visual>
+    </link>
+    <link name="01_FlatSprocket">
+        <visual>
+            <origin xyz="-0.55 0.0 -0.47" rpy="1.570795 0.0 0.0"/>
+            <geometry>
+                <mesh filename="package://ixnaminki_description/meshes/ASSY_TrenInferior/FlatSprocket.STL" scale="0.004 0.004 0.004"/>
+            </geometry>
+        </visual>
+    </link>
+    <link name="02_FlatSprocket">
+        <visual>
+            <origin xyz="-0.55 0.0 -0.47" rpy="1.570795 0.0 0.0"/>
+            <geometry>
+                <mesh filename="package://ixnaminki_description/meshes/ASSY_TrenInferior/FlatSprocket.STL" scale="0.004 0.004 0.004"/>
             </geometry>
         </visual>
@@ -107,8 +147,42 @@
         <parent link="02_EjePrincipal2"/>
         <child link = "01_Placa"/>
-        <origin xyz="0.0 0.0 0.0"/>
+        <origin xyz="-0.69 1.0 0.28"/>
         <axis xyz="0 1 0"/>
         <limit lower="-1.570795" upper="1.570795"
                effort="${effort}" velocity="${velocity}"/>
     </joint>
+    <joint name ="joint_8" type="revolute">
+        <parent link="02_EjePrincipal2"/>
+        <child link = "02_Placa"/>
+        <origin xyz="-0.69 -1.0 0.28"/>
+        <axis xyz="0 1 0"/>
+        <limit lower="-1.570795" upper="1.570795"
+               effort="${effort}" velocity="${velocity}"/>
+    </joint>
+    <joint name ="joint_9" type="revolute">
+        <parent link="02_EjePrincipal"/>
+        <child link = "03_Placa"/>
+        <origin xyz="0.84 1.0 0.29"/>
+        <axis xyz="0 1 0"/>
+        <limit lower="-1.570795" upper="1.570795"
+               effort="${effort}" velocity="${velocity}"/>
+    </joint>
+    <joint name ="joint_10" type="revolute">
+        <parent link="02_EjePrincipal"/>
+        <child link = "04_Placa"/>
+        <origin xyz="0.84 -1.0 0.29"/>
+        <axis xyz="0 1 0"/>
+        <limit lower="-1.570795" upper="1.570795"
+               effort="${effort}" velocity="${velocity}"/>
+    </joint>
+    <joint name="joint_11" type="fixed">
+        <origin xyz="-0.69 -0.015 0.28" rpy="0.0 0.0 0.0"/>
+        <parent link="01_Placa"/>
+        <child link="01_FlatSprocket"/>
+    </joint>
+    <joint name="joint_12" type="fixed">
+        <origin xyz="-0.69 0.015 0.28" rpy="0.0 0.0 0.0"/>
+        <parent link="02_Placa"/>
+        <child link="02_FlatSprocket"/>
+    </joint>
 </robot>

Commit message: parte 1 terminada

File: ixnaminki_description/urdf/ixnaminki_des.urdf.xacro (robot description, xacro)
@@ -109,4 +109,20 @@
         </visual>
     </link>
+    <link name="03_FlatSprocket">
+        <visual>
+            <origin xyz="0.01 0.0 -0.492" rpy="1.570795 0.0 0.0"/>
+            <geometry>
+                <mesh filename="package://ixnaminki_description/meshes/ASSY_TrenInferior/FlatSprocket.STL" scale="0.004 0.004 0.004"/>
+            </geometry>
+        </visual>
+    </link>
+    <link name="04_FlatSprocket">
+        <visual>
+            <origin xyz="0.01 0.0 -0.492" rpy="1.570795 0.0 0.0"/>
+            <geometry>
+                <mesh filename="package://ixnaminki_description/meshes/ASSY_TrenInferior/FlatSprocket.STL" scale="0.004 0.004 0.004"/>
+            </geometry>
+        </visual>
+    </link>
     <joint name="virtual_joint" type="fixed">
         <parent link="world"/>
@@ -186,3 +202,13 @@
         <child link="02_FlatSprocket"/>
     </joint>
+    <joint name="joint_13" type="fixed">
+        <origin xyz="0.84 -0.015 0.29" rpy="0.0 0.0 0.0"/>
+        <parent link="03_Placa"/>
+        <child link="03_FlatSprocket"/>
+    </joint>
+    <joint name="joint_14" type="fixed">
+        <origin xyz="0.84 0.015 0.29" rpy="0.0 0.0 0.0"/>
+        <parent link="04_Placa"/>
+        <child link="04_FlatSprocket"/>
+    </joint>
 </robot>

Commit message: Insersión del brazo

File: ixnaminki_description/urdf/ixnaminki_des.urdf.xacro (robot description, xacro)
@@ -5,4 +5,5 @@
     <xacro:property name="velocity" value="10.0" />
     <link name="world"/>
+<!-- CUERPO -->
     <link name="base_link">
         <visual>
@@ -19,4 +20,7 @@
                 <mesh filename="package://ixnaminki_description/meshes/ASSY_TrenInferior/02_EjePrincipal.STL" scale="0.004 0.004 0.004"/>
             </geometry>
+            <material name="base">
+                <color rgba="0.73 0.65 0.69 0.8"/>
+            </material>
         </visual>
     </link>
@@ -27,4 +31,7 @@
                 <mesh filename="package://ixnaminki_description/meshes/ASSY_TrenInferior/02_EjePrincipal.STL" scale="0.004 0.004 0.004"/>
             </geometry>
+            <material name="base">
+                <color rgba="0.73 0.65 0.69 0.8"/>
+            </material>
         </visual>
     </link>
@@ -212,3 +219,71 @@
         <child link="04_FlatSprocket"/>
     </joint>
+<!-- BRAZO -->
+    <link name="base_link_arm">
+        <visual>
+            <origin xyz="0.0 0.0 0.0" rpy="1.570795 0.0 0.0"/>
+            <geometry>
+                <mesh filename="package://ixnaminki_description/meshes/BRAZO/base_002.STL" scale="0.004 0.004 0.004"/>
+            </geometry>
+            <material name="base2">
+                <color rgba="1.0 0.0 1.0 1.0"/>
+            </material>
+        </visual>
+    </link>
+    <link name="rotation_base">
+        <visual>
+            <origin xyz="-0.27 -0.26 0.0" rpy="1.570795 0.0 1.570795"/>
+            <geometry>
+                <mesh filename="package://ixnaminki_description/meshes/BRAZO/base_004.STL" scale="0.004 0.004 0.004"/>
+            </geometry>
+            <material name="base3">
+                <color rgba="0.40 0.211 0.72 0.46"/>
+            </material>
+        </visual>
+    </link>
+    <link name="01_oreja">
+        <visual>
+            <origin xyz="0.0 0.0 0.0" rpy="1.570795 0.0 0.0"/>
+            <geometry>
+                <mesh filename="package://ixnaminki_description/meshes/BRAZO/Orejas.STL" scale="0.004 0.004 0.004"/>
+            </geometry>
+            <material name="base3">
+                <color rgba="0.40 0.211 0.72 0.46"/>
+            </material>
+        </visual>
+    </link>
+    <link name="02_oreja">
+        <visual>
+            <origin xyz="0.0 0.0 0.0" rpy="1.570795 0.0 0.0"/>
+            <geometry>
+                <mesh filename="package://ixnaminki_description/meshes/BRAZO/Orejas.STL" scale="0.004 0.004 0.004"/>
+            </geometry>
+            <material name="base3">
+                <color rgba="0.40 0.211 0.72 0.46"/>
+            </material>
+        </visual>
+    </link>
+    <joint name="joint_15" type="fixed">
+        <origin xyz="0.1 0.25 0.55" rpy="0.0 0.0 0.0"/>
+        <parent link="base_link"/>
+        <child link="base_link_arm"/>
+    </joint>
+    <joint name ="joint_16" type="revolute">
+        <parent link="base_link_arm"/>
+        <child link = "rotation_base"/>
+        <origin xyz="0.29 -0.29 0.05"/>
+        <axis xyz="0 0 1"/>
+        <limit lower="-1.570795" upper="1.570795"
+               effort="${effort}" velocity="${velocity}"/>
+    </joint>
+    <joint name="joint_17" type="fixed">
+        <origin xyz="-0.15 0.15 0.25" rpy="1.570795 0.0 0.0"/>
+        <parent link="rotation_base"/>
+        <child link="01_oreja"/>
+    </joint>
+    <joint name="joint_18" type="fixed">
+        <origin xyz="-0.15 -0.15 0.25" rpy="1.570795 0.0 0.0"/>
+        <parent link="rotation_base"/>
+        <child link="02_oreja"/>
+    </joint>
 </robot>

Commit message: Finalizado

File: ixnaminki_description/urdf/ixnaminki_des.urdf.xacro (robot description, xacro)
@@ -12,4 +12,7 @@
                 <mesh filename="package://ixnaminki_description/meshes/ASSY_TrenInferior/01_Chasis.STL" scale="0.004 0.004 0.004"/>
             </geometry>
+            <material name="base00">
+                <color rgba="0.5 0.3 0.2 0.8"/>
+            </material>
         </visual>
     </link>
@@ -42,4 +45,5 @@
                 <mesh filename="package://ixnaminki_description/meshes/ASSY_TrenInferior/PlateSprocket.STL" scale="0.004 0.004 0.004"/>
             </geometry>
+            <material name="base"/>
         </visual>
     </link>
@@ -50,4 +54,5 @@
                 <mesh filename="package://ixnaminki_description/meshes/ASSY_TrenInferior/PlateSprocket.STL" scale="0.004 0.004 0.004"/>
             </geometry>
+            <material name="base"/>
         </visual>
     </link>
@@ -58,4 +63,5 @@
                 <mesh filename="package://ixnaminki_description/meshes/ASSY_TrenInferior/PlateSprocket.STL" scale="0.004 0.004 0.004"/>
             </geometry>
+            <material name="base"/>
         </visual>
     </link>
@@ -66,4 +72,5 @@
                 <mesh filename="package://ixnaminki_description/meshes/ASSY_TrenInferior/PlateSprocket.STL" scale="0.004 0.004 0.004"/>
             </geometry>
+            <material name="base"/>
         </visual>
     </link>
@@ -106,4 +113,5 @@
                 <mesh filename="package://ixnaminki_description/meshes/ASSY_TrenInferior/FlatSprocket.STL" scale="0.004 0.004 0.004"/>
             </geometry>
+            <material name="base"/>
         </visual>
     </link>
@@ -114,4 +122,5 @@
                 <mesh filename="package://ixnaminki_description/meshes/ASSY_TrenInferior/FlatSprocket.STL" scale="0.004 0.004 0.004"/>
             </geometry>
+            <material name="base"/>
         </visual>
     </link>
@@ -122,4 +131,5 @@
                 <mesh filename="package://ixnaminki_description/meshes/ASSY_TrenInferior/FlatSprocket.STL" scale="0.004 0.004 0.004"/>
             </geometry>
+            <material name="base"/>
         </visual>
     </link>
@@ -130,4 +140,5 @@
                 <mesh filename="package://ixnaminki_description/meshes/ASSY_TrenInferior/FlatSprocket.STL" scale="0.004 0.004 0.004"/>
             </geometry>
+            <material name="base"/>
         </visual>
     </link>
@@ -261,4 +272,114 @@
             <material name="base3">
                 <color rgba="0.40 0.211 0.72 0.46"/>
+            </material>
+        </visual>
+    </link>
+    <link name="eje_brazo">
+        <visual>
+            <origin xyz="0.0 0.0 0.0" rpy="1.570795 0.0 0.0"/>
+            <geometry>
+                <mesh filename="package://ixnaminki_description/meshes/BRAZO/eje20mm.STL" scale="0.004 0.004 0.004"/>
+            </geometry>
+            <material name="base4">
+                <color rgba="0.0 0.0 0.0 0.5"/>
+            </material>
+        </visual>
+    </link>
+    <link name="placa_baja_brazo_izquierdo">
+        <visual>
+            <origin xyz="0.05 -0.1 -0.15" rpy="0.0 -1.04719 0.0"/>
+            <geometry>
+                <mesh filename="package://ixnaminki_description/meshes/BRAZO/Brazo.STL" scale="0.004 0.004 0.004"/>
+            </geometry>
+            <material name="base5">
+                <color rgba="1 0.0 0.3 0.9"/>
+            </material>
+        </visual>
+    </link>
+    <link name="placa_baja_brazo_derecho">
+        <visual>
+            <origin xyz="0.05 -0.05 -0.15" rpy="0.0 -1.04719 0.0"/>
+            <geometry>
+                <mesh filename="package://ixnaminki_description/meshes/BRAZO/BrazoB.STL" scale="0.004 0.004 0.004"/>
+            </geometry>
+            <material name="base5">
+                <color rgba="1 0.0 0.3 0.9"/>
+            </material>
+        </visual>
+    </link>
+    <link name="carcasa">
+        <visual>
+            <origin xyz="0.0 -0.11 0.0" rpy="0.5 0.0 1.570795"/>
+            <geometry>
+                <mesh filename="package://ixnaminki_description/meshes/BRAZO/Carcasa.STL" scale="0.005 0.004 0.004"/>
+            </geometry>
+            <material name="base6">
+                <color rgba="0.0 0.0 0.2 0.67"/>
+            </material>
+        </visual>
+    </link>
+    <link name="placa_alta_brazo_izquierdo">
+        <visual>
+            <origin xyz="-0.15 -0.045 -0.11" rpy="1.570795 0.0 0.0"/>
+            <geometry>
+                <mesh filename="package://ixnaminki_description/meshes/BRAZO/Brazo2A.STL" scale="0.005 0.004 0.004"/>
+            </geometry>
+            <material name="base7">
+                <color rgba="0.0 0.0 0.7 0.98"/>
+            </material>
+        </visual>
+    </link>
+    <link name="placa_alta_brazo_derecho">
+        <visual>
+            <origin xyz="-0.15 -0.445 -0.11" rpy="1.570795 0.0 0.0"/>
+            <geometry>
+                <mesh filename="package://ixnaminki_description/meshes/BRAZO/Brazo2A.STL" scale="0.005 0.004 0.004"/>
+            </geometry>
+            <material name="base7">
+                <color rgba="0.0 0.0 0.7 0.98"/>
+            </material>
+        </visual>
+    </link>
+    <link name="01_espaciador">
+        <visual>
+            <origin xyz="0.05 -0.07 0.05" rpy="0.0 0.0 -1.570795"/>
+            <geometry>
+                <mesh filename="package://ixnaminki_description/meshes/BRAZO/espaciador.STL" scale="0.005 0.004 0.004"/>
+            </geometry>
+            <material name="base8">
+                <color rgba="0.0 0.0 0.0 1"/>
+            </material>
+        </visual>
+    </link>
+    <link name="02_espaciador">
+        <visual>
+            <origin xyz="-0.05 -0.07 0.05" rpy="0.0 0.0 -1.570795"/>
+            <geometry>
+                <mesh filename="package://ixnaminki_description/meshes/BRAZO/espaciador.STL" scale="0.005 0.004 0.004"/>
+            </geometry>
+            <material name="base8">
+                <color rgba="0.0 0.0 0.0 1"/>
+            </material>
+        </visual>
+    </link>
+    <link name="03_espaciador">
+        <visual>
+            <origin xyz="0.05 -0.07 -0.05" rpy="0.0 0.0 -1.570795"/>
+            <geometry>
+                <mesh filename="package://ixnaminki_description/meshes/BRAZO/espaciador.STL" scale="0.005 0.004 0.004"/>
+            </geometry>
+            <material name="base8">
+                <color rgba="0.0 0.0 0.0 1"/>
+            </material>
+        </visual>
+    </link>
+    <link name="04_espaciador">
+        <visual>
+            <origin xyz="-0.05 -0.07 -0.05" rpy="0.0 0.0 -1.570795"/>
+            <geometry>
+                <mesh filename="package://ixnaminki_description/meshes/BRAZO/espaciador.STL" scale="0.005 0.004 0.004"/>
+            </geometry>
+            <material name="base8">
+                <color rgba="0.0 0.0 0.0 1"/>
             </material>
         </visual>
@@ -287,3 +408,65 @@
         <child link="02_oreja"/>
     </joint>
+    <joint name="joint_19" type="fixed">
+        <origin xyz="-0.05 0.25 0.14" rpy="0.0 0.0 0.0"/>
+        <parent link="rotation_base"/>
+        <child link="eje_brazo"/>
+    </joint>
+    <joint name ="joint_20" type="revolute">
+        <parent link="eje_brazo"/>
+        <child link = "placa_baja_brazo_izquierdo"/>
+        <origin xyz="0.03 0.0 0.03"/>
+        <axis xyz="0 1 0"/>
+        <limit lower="-1.570795" upper="0.909"
+               effort="${effort}" velocity="${velocity}"/>
+    </joint>
+    <joint name ="joint_21" type="revolute">
+        <parent link="eje_brazo"/>
+        <child link = "placa_baja_brazo_derecho"/>
+        <origin xyz="0.03 -0.44 0.03"/>
+        <axis xyz="0 1 0"/>
+        <limit lower="-1.570795" upper="0.909"
+               effort="${effort}" velocity="${velocity}"/>
+    </joint>
+    <joint name="joint_22" type="fixed">
+        <origin xyz="1.0 -0.32 1.3" rpy="0.0 0.0 0.0"/>
+        <parent link="placa_baja_brazo_izquierdo"/>
+        <child link="carcasa"/>
+    </joint>
+    <joint name ="joint_23" type="revolute">
+        <parent link="placa_baja_brazo_derecho"/>
+        <child link = "placa_alta_brazo_izquierdo"/>
+        <origin xyz="0.91 0.0 1.65"/>
+        <axis xyz="0 1 0"/>
+        <limit lower="-3.0" upper="3.0"
+               effort="${effort}" velocity="${velocity}"/>
+    </joint>
+    <joint name ="joint_24" type="revolute">
+        <parent link="placa_baja_brazo_derecho"/>
+        <child link = "placa_alta_brazo_derecho"/>
+        <origin xyz="0.91 0.0 1.65"/>
+        <axis xyz="0 1 0"/>
+        <limit lower="-3.0" upper="3.0"
+               effort="${effort}" velocity="${velocity}"/>
+    </joint>
+    <joint name="joint_25" type="fixed">
+        <origin xyz="0.0 0.0 0.0" rpy="0.0 0.0 0.0"/>
+        <parent link="placa_alta_brazo_derecho"/>
+        <child link="01_espaciador"/>
+    </joint>
+    <joint name="joint_26" type="fixed">
+        <origin xyz="0.0 0.0 0.0" rpy="0.0 0.0 0.0"/>
+        <parent link="placa_alta_brazo_derecho"/>
+        <child link="02_espaciador"/>
+    </joint>
+    <joint name="joint_27" type="fixed">
+        <origin xyz="0.0 0.0 0.0" rpy="0.0 0.0 0.0"/>
+        <parent link="placa_alta_brazo_derecho"/>
+        <child link="03_espaciador"/>
+    </joint>
+    <joint name="joint_28" type="fixed">
+        <origin xyz="0.0 0.0 0.0" rpy="0.0 0.0 0.0"/>
+        <parent link="placa_alta_brazo_derecho"/>
+        <child link="04_espaciador"/>
+    </joint>
 </robot>
